Commit message: updates

File: legged_unitree/legged_unitree_description/urdf/a1/const.xacro (robot description, xacro)
@@ -4,30 +4,28 @@
     <xacro:property name="stick_mass" value="0.00001"/>
     <!-- simplified collision value -->
-    <xacro:property name="PI" value="3.1415926535897931"/>
-    <xacro:property name="body_center_x" value="0.0"/>
-    <xacro:property name="body_center_y" value="0.0"/>
-    <xacro:property name="body_center_z" value="0.0"/>
-    <xacro:property name="trunk_width" value="0.350"/>
-    <xacro:property name="trunk_length" value="0.57"/>
-    <xacro:property name="trunk_height" value="0.149"/>
-    <xacro:property name="hip_radius" value="0.050"/>
-    <xacro:property name="hip_length" value="0.06"/>
-    <xacro:property name="thigh_width" value="0.0374"/>
-    <xacro:property name="thigh_height" value="0.043"/>
-    <xacro:property name="calf_width" value="0.0208"/>
+    <xacro:property name="trunk_width" value="0.194"/>
+    <xacro:property name="trunk_length" value="0.267"/>
+    <xacro:property name="trunk_height" value="0.114"/>
+    <xacro:property name="hip_radius" value="0.046"/>
+    <xacro:property name="hip_length" value="0.04"/>
+    <xacro:property name="thigh_shoulder_radius" value="0.041"/>
+    <xacro:property name="thigh_shoulder_length" value="0.04"/>
+    <xacro:property name="thigh_shoulder_y_offset" value="-0.008"/>
+    <xacro:property name="thigh_width" value="0.03"/>
+    <xacro:property name="thigh_height" value="0.034"/>
+    <xacro:property name="thigh_x_offset" value="-0.015"/>
+    <xacro:property name="calf_width" value="0.016"/>
     <xacro:property name="calf_height" value="0.016"/>
-    <xacro:property name="foot_radius" value="0.0265"/>
-    <xacro:property name="stick_radius" value="0.01"/>
-    <xacro:property name="stick_length" value="0.2"/>
+    <xacro:property name="calf_x_offset" value="0.0"/>
+    <xacro:property name="foot_radius" value="0.02"/>
     <!-- kinematic value -->
-    <xacro:property name="thigh_offset" value="0.02"/>
-    <xacro:property name="thigh_length" value="0.201"/>
-    <xacro:property name="calf_length" value="0.230"/>
+    <xacro:property name="thigh_offset" value="0.0838"/>
+    <xacro:property name="thigh_length" value="0.2"/>
+    <xacro:property name="calf_length" value="0.2"/>
     <!-- leg offset from trunk center value -->
-    <xacro:property name="leg_offset_x" value="${0.135}"/>
-    <xacro:property name="leg_offset_y" value="${0.057}"/>
-    <xacro:property name="leg_offset_z" value="${0.024}"/>
+    <xacro:property name="leg_offset_x" value="0.1805"/>
+    <xacro:property name="leg_offset_y" value="0.047"/>
     <xacro:property name="trunk_offset_z" value="0.01675"/>
-    <xacro:property name="hip_offset" value="0.083"/>
+    <xacro:property name="hip_offset" value="0.065"/>
     <!-- joint limits -->
     <xacro:property name="damping" value="0"/>
@@ -48,56 +46,47 @@
     <!-- trunk -->
     <xacro:property name="trunk_mass" value="6.0"/>
-    <xacro:property name="trunk_com_x" value="0.02"/>
-    <xacro:property name="trunk_com_y" value="0.00194"/>
-    <xacro:property name="trunk_com_z" value="0.0"/>
+    <xacro:property name="trunk_com_x" value="0.0000"/>
+    <xacro:property name="trunk_com_y" value="0.0041"/>
+    <xacro:property name="trunk_com_z" value="-0.0005"/>
     <xacro:property name="trunk_ixx" value="0.0158533"/>
-    <xacro:property name="trunk_ixy" value="-0.0001332"/>
-    <xacro:property name="trunk_ixz" value="-0.0002403"/>
-    <xacro:property name="trunk_iyy" value="0.04168"/>
-    <xacro:property name="trunk_iyz" value="0.000015299"/>
-    <xacro:property name="trunk_izz" value="0.04742"/>
+    <xacro:property name="trunk_ixy" value="-0.0000366"/>
+    <xacro:property name="trunk_ixz" value="-0.0000611"/>
+    <xacro:property name="trunk_iyy" value="0.0377999"/>
+    <xacro:property name="trunk_iyz" value="-0.0000275"/>
+    <xacro:property name="trunk_izz" value="0.0456542"/>
     <!-- hip (left front) -->
-    <xacro:property name="hip_mass" value="0.599"/>
-    <xacro:property name="hip_com_x" value="-0.011957"/>
-    <xacro:property name="hip_com_y" value="0.000306"/>
-    <xacro:property name="hip_com_z" value="0.000366"/>
-    <xacro:property name="hip_ixx" value="0.0004159"/>
-    <xacro:property name="hip_ixy" value="0.000004253"/>
-    <xacro:property name="hip_ixz" value="0.000000368"/>
-    <xacro:property name="hip_iyy" value="0.0007108"/>
-    <xacro:property name="hip_iyz" value="0.000000215"/>
-    <xacro:property name="hip_izz" value="0.0004707"/>
+    <xacro:property name="hip_mass" value="0.595"/>
+    <xacro:property name="hip_com_x" value="-0.003875"/>
+    <xacro:property name="hip_com_y" value="0.001622"/>
+    <xacro:property name="hip_com_z" value="0.000042"/>
+    <xacro:property name="hip_ixx" value="0.000402747"/>
+    <xacro:property name="hip_ixy" value="-0.000008709"/>
+    <xacro:property name="hip_ixz" value="-0.000000297"/>
+    <xacro:property name="hip_iyy" value="0.000691123"/>
+    <xacro:property name="hip_iyz" value="-0.000000545"/>
+    <xacro:property name="hip_izz" value="0.000487919"/>
     <!-- thigh -->
-    <xacro:property name="thigh_mass" value="1.080"/>
-    <xacro:property name="thigh_com_x" value="-0.000684"/>
-    <xacro:property name="thigh_com_y" value="-0.010999"/>
-    <xacro:property name="thigh_com_z" value="-0.035487"/>
-    <xacro:property name="thigh_ixx" value="0.005666803"/>
-    <xacro:property name="thigh_ixy" value="0.000003597"/>
-    <xacro:property name="thigh_ixz" value="0.000491446"/>
-    <xacro:property name="thigh_iyy" value="0.005847229"/>
-    <xacro:property name="thigh_iyz" value="0.000010086"/>
-    <xacro:property name="thigh_izz" value="0.000369811"/>
+    <xacro:property name="thigh_mass" value="0.888"/>
+    <xacro:property name="thigh_com_x" value="-0.003574"/>
+    <xacro:property name="thigh_com_y" value="-0.019529"/>
+    <xacro:property name="thigh_com_z" value="-0.030323"/>
+    <xacro:property name="thigh_ixx" value="0.005251806"/>
+    <xacro:property name="thigh_ixy" value="-0.000002168"/>
+    <xacro:property name="thigh_ixz" value="0.000346889"/>
+    <xacro:property name="thigh_iyy" value="0.005000475"/>
+    <xacro:property name="thigh_iyz" value="-0.000028174"/>
+    <xacro:property name="thigh_izz" value="0.001110200"/>
     <!-- calf -->
-    <xacro:property name="calf_mass" value="0.265"/>
-    <xacro:property name="calf_com_x" value="0.000252"/>
-    <xacro:property name="calf_com_y" value="0.000194"/>
-    <xacro:property name="calf_com_z" value="-0.05192"/>
-    <xacro:property name="calf_ixx" value="0.0004583"/>
-    <xacro:property name="calf_ixy" value="-0.000000095"/>
-    <xacro:property name="calf_ixz" value="0.000026512"/>
-    <xacro:property name="calf_iyy" value="0.0004675"/>
-    <xacro:property name="calf_iyz" value="0.000000277"/>
-    <xacro:property name="calf_izz" value="0.000029145"/>
+    <xacro:property name="calf_mass" value="0.151"/>
+    <xacro:property name="calf_com_x" value="0.007105"/>
+    <xacro:property name="calf_com_y" value="-0.000239"/>
+    <xacro:property name="calf_com_z" value="-0.096933"/>
+    <xacro:property name="calf_ixx" value="0.002344758"/>
+    <xacro:property name="calf_ixy" value="0.0"/>
+    <xacro:property name="calf_ixz" value="-0.000141275"/>
+    <xacro:property name="calf_iyy" value="0.002360755"/>
+    <xacro:property name="calf_iyz" value="0.0"/>
+    <xacro:property name="calf_izz" value="0.000031158"/>
     <!-- foot -->
-    <xacro:property name="foot_mass" value="0.078"/>
-    <xacro:property name="foot_com_x" value="-0.007246"/>
-    <xacro:property name="foot_com_y" value="0.000092"/>
-    <xacro:property name="foot_com_z" value="-0.038267"/>
-    <xacro:property name="foot_ixx" value="0.000029902"/>
-    <xacro:property name="foot_ixy" value="-0.000000022"/>
-    <xacro:property name="foot_ixz" value="-0.000004427"/>
-    <xacro:property name="foot_iyy" value="0.000030583"/>
-    <xacro:property name="foot_iyz" value="-0.000000099"/>
-    <xacro:property name="foot_izz" value="0.000014025"/>
+    <xacro:property name="foot_mass" value="0.06"/>
 </robot>

File: legged_unitree/legged_unitree_description/urdf/aliengo/const.xacro (robot description, xacro)
@@ -12,15 +12,14 @@
     <xacro:property name="thigh_shoulder_length" value="0.03"/>
     <xacro:property name="thigh_shoulder_y_offset" value="0.0"/>
-    <xacro:property name="thigh_x_offset" value="0.0"/>
     <xacro:property name="thigh_width" value="0.0374"/>
     <xacro:property name="thigh_height" value="0.043"/>
-    <xacro:property name="calf_width" value="0.0208"/>
-    <xacro:property name="calf_height" value="0.016"/>
+    <xacro:property name="thigh_x_offset" value="-0.015"/>
+    <xacro:property name="calf_width" value="0.04"/>
+    <xacro:property name="calf_height" value="0.03"/>
+    <xacro:property name="calf_x_offset" value="0.008"/>
     <xacro:property name="foot_radius" value="0.0265"/>
-    <xacro:property name="stick_radius" value="0.01"/>
-    <xacro:property name="stick_length" value="0.2"/>
     <!-- kinematic value -->
-    <xacro:property name="thigh_offset" value="0.02"/><!-- decalage lateral HIP -> upper_leg - lateral difference between HIP and upper_leg -->
-    <xacro:property name="thigh_length" value="0.201"/><!-- upper leg size, from HIP axis, to lower leg axis-->
+    <xacro:property name="thigh_offset" value="0.0868"/>
+    <xacro:property name="thigh_length" value="0.25"/>
     <xacro:property name="calf_length" value="0.25"/>
     <!-- leg offset from trunk center value -->

File: legged_unitree/legged_unitree_description/urdf/common/leg.xacro (robot description, xacro)
@@ -21,17 +21,17 @@
             <visual>
                 <xacro:if value="${(mirror_dae == True) and (front_hind_dae == True)}">
-                    <origin rpy="0 0 0" xyz="-0.055 0 0"/>
+                    <origin rpy="0 0 0" xyz="0 0 0"/>
                 </xacro:if>
                 <xacro:if value="${(mirror_dae == False) and (front_hind_dae == True)}">
-                    <origin rpy="${PI} 0 0" xyz="-0.055 0 0"/>
+                    <origin rpy="${pi} 0 0" xyz="0 0 0"/>
                 </xacro:if>
                 <xacro:if value="${(mirror_dae == True) and (front_hind_dae == False)}">
-                    <origin rpy="0 ${PI} 0" xyz="0.055 0 0"/>
+                    <origin rpy="0 ${pi} 0" xyz="0 0 0"/>
                 </xacro:if>
                 <xacro:if value="${(mirror_dae == False) and (front_hind_dae == False)}">
-                    <origin rpy="${PI} ${PI} 0" xyz="0.055 0 0"/>
+                    <origin rpy="${pi} ${pi} 0" xyz="0 0 0"/>
                 </xacro:if>
                 <geometry>
-                    <mesh filename="package://legged_unitree_description/meshes/a1/leg/textured/ylo2texturedhip.dae"
+                    <mesh filename="package://legged_unitree_description/meshes/$(arg robot_type)/hip.dae"
                           scale="1 1 1"/>
                 </geometry>
@@ -54,5 +54,5 @@
         </link>
         <joint name="${prefix}_HFE" type="revolute">
-            <origin rpy="0 ${PI/2.0} 0" xyz="${thigh_width-0.0374} ${thigh_offset*mirror} 0"/>
+            <origin rpy="0 0 0" xyz="0 ${thigh_offset*mirror} 0"/>
             <parent link="${prefix}_hip"/>
             <child link="${prefix}_thigh"/>
@@ -67,10 +67,10 @@
                 <geometry>
                     <xacro:if value="${mirror_dae == True}">
-                        <mesh filename="package://legged_unitree_description/meshes/a1/leg/textured/ylo2_textured_upper_leg.dae"
+                        <mesh filename="package://legged_unitree_description/meshes/$(arg robot_type)/thigh.dae"
                               scale="1 1 1"/>
                     </xacro:if>
                     <xacro:if value="${mirror_dae == False}">
-                        <mesh filename="package://legged_unitree_description/meshes/a1/leg/textured/ylo2_textured_upper_leg.dae"
-                              scale="1 -1 1"/>
+                        <mesh filename="package://legged_unitree_description/meshes/$(arg robot_type)/thigh_mirror.dae"
+                              scale="1 1 1"/>
                     </xacro:if>
                 </geometry>
@@ -78,7 +78,13 @@
             </visual>
             <collision>
-                <origin rpy="0 ${PI/2.0} 0" xyz="0 0 ${-thigh_length/2.0}"/>
+                <origin rpy="0 ${pi/2.0+0.1} 0" xyz="${thigh_x_offset} 0 ${-thigh_length/2.0}"/>
                 <geometry>
                     <box size="${thigh_length} ${thigh_width} ${thigh_height}"/>
+                </geometry>
+            </collision>
+            <collision>
+                <origin rpy="${pi/2.0} 0 0" xyz="0 ${mirror*thigh_shoulder_y_offset} 0"/>
+                <geometry>
+                    <cylinder length="${thigh_shoulder_length}" radius="${thigh_shoulder_radius}"/>
                 </geometry>
             </collision>
@@ -93,5 +99,5 @@
         </link>
         <joint name="${prefix}_KFE" type="revolute">
-            <origin rpy="0 ${-PI} 0" xyz="-0.001 ${(0.075*mirror)} ${-thigh_length}"/>
+            <origin rpy="0 0 0" xyz="0 0 ${-thigh_length}"/>
             <parent link="${prefix}_thigh"/>
             <child link="${prefix}_calf"/>
@@ -104,5 +110,5 @@
                 <origin rpy="0 0 0" xyz="0 0 0"/>
                 <geometry>
-                    <mesh filename="package://legged_unitree_description/meshes/a1/leg/textured/lower_leg.dae"
+                    <mesh filename="package://legged_unitree_description/meshes/$(arg robot_type)/calf.dae"
                           scale="1 1 1"/>
                 </geometry>
@@ -110,8 +116,7 @@
             </visual>
             <collision>
-                <origin rpy="0 ${PI/2.0} 0" xyz="0 0 ${-calf_length/2.0}"/>
+                <origin rpy="0 ${pi/2.0} 0" xyz="${calf_x_offset} 0 ${-calf_length/2.0}"/>
                 <geometry>
-                    <mesh filename="package://legged_unitree_description/meshes/a1/leg/fl_lower_leg_collision.stl"
-                          scale="1 1 1"/>
+                    <box size="${calf_length} ${calf_width} ${calf_height}"/>
                 </geometry>
             </collision>
@@ -132,15 +137,14 @@
         <link name="${prefix}_FOOT">
             <visual>
-                <origin rpy="0 0 0" xyz="0.009 ${(0.001*mirror)+0.001} 0.069"/>
+                <origin rpy="0 0 0" xyz="0 0 0"/>
                 <geometry>
-                    <mesh filename="package://legged_unitree_description/meshes/a1/leg/fl_foot.dae"
-                          scale="1 1 1"/>
+                    <sphere radius="${foot_radius-0.01}"/>
                 </geometry>
                 <material name="orange"/>
             </visual>
             <collision>
-                <origin rpy="0 0 0" xyz="0.009 ${(0.001*mirror)+0.001} 0.069"/>
+                <origin rpy="0 0 0" xyz="0 0 0"/>
                 <geometry>
-                    <mesh filename="package://legged_unitree_description/meshes/a1/legfh/fl_foot.dae" scale="1.0 1.0 1.0"/>-->
+                    <sphere radius="${foot_radius}"/>
                 </geometry>
             </collision>
@@ -156,4 +160,30 @@
             <disableFixedJointLumping>true</disableFixedJointLumping>
         </gazebo>
+        <gazebo reference="${prefix}_hip">
+            <mu1>0.2</mu1>
+            <mu2>0.2</mu2>
+            <material>Gazebo/DarkGrey</material>
+        </gazebo>
+        <gazebo reference="${prefix}_thigh">
+            <mu1>0.2</mu1>
+            <mu2>0.2</mu2>
+            <self_collide>0</self_collide>
+            <material>Gazebo/DarkGrey</material>
+            <kp value="1000000.0"/>
+            <kd value="100.0"/>
+        </gazebo>
+        <gazebo reference="${prefix}_calf">
+            <mu1>0.6</mu1>
+            <mu2>0.6</mu2>
+            <self_collide>1</self_collide>
+        </gazebo>
+        <gazebo reference="${prefix}_FOOT">
+            <mu1>0.6</mu1>
+            <mu2>0.6</mu2>
+            <self_collide>1</self_collide>
+            <material>Gazebo/DarkGrey</material>
+            <kp value="1000000.0"/>
+            <kd value="100.0"/>
+        </gazebo>
         <xacro:leg_transmission name="${prefix}"/>
     </xacro:macro>

File: legged_unitree/legged_unitree_description/urdf/robot.xacro (robot description, xacro)
@@ -9,11 +9,11 @@
     <link name="base">
         <visual>
-            <origin rpy="0 0 0" xyz="${body_center_x} ${body_center_y} ${body_center_z}"/>
+            <origin rpy="0 0 0" xyz="0 0 0"/>
             <geometry>
-                <mesh filename="package://legged_unitree_description/meshes/a1/body/textured/ylo2_textured_body.dae" scale="1 1 1"/>
+                <mesh filename="package://legged_unitree_description/meshes/$(arg robot_type)/trunk.dae" scale="1 1 1"/>
             </geometry>
         </visual>
         <collision>
-            <origin rpy="0 0 0" xyz="${body_center_x} ${body_center_y} ${body_center_z}"/>
+            <origin rpy="0 0 0" xyz="0 0 0"/>
             <geometry>
                 <box size="${trunk_length} ${trunk_width} ${trunk_height}"/>
@@ -29,86 +29,16 @@
         </inertial>
     </link>
-    <joint name="abad_motors_joint" type="fixed">
-        <parent link="base"/>
-        <child link="abad_motors"/>
-        <origin rpy="0 0 0" xyz="0 0 0"/>
-    </joint>
-    <link name="abad_motors">
-        <visual>
-            <origin rpy="0 0 0" xyz="${body_center_x} ${body_center_y} ${body_center_z}"/>
-            <geometry>
-                <mesh filename="package://legged_unitree_description/meshes/a1/body/textured/ylo2_textured_abad_motors.dae" scale="1 1 1"/>
-            </geometry>
-            <material name="white"/>
-        </visual>
-    </link>
-    <joint name="covers_joint" type="fixed">
-        <parent link="base"/>
-        <child link="covers"/>
-        <origin rpy="0 0 0" xyz="0 0 0"/>
-    </joint>
-    <link name="covers">
-        <visual>
-            <origin rpy="0 0 0" xyz="${body_center_x} ${body_center_y} ${body_center_z}"/>
-            <geometry>
-                <mesh filename="package://legged_unitree_description/meshes/a1/body/textured/ylo2_textured_cover.dae" scale="1 1 1"/>
-            </geometry>
-            <material name="orange"/>
-        </visual>
-    </link>
-    <joint name="accessories_joint" type="fixed">
-        <parent link="base"/>
-        <child link="accessories"/>
-        <origin rpy="0 0 0" xyz="0 0 0"/>
-    </joint>
-    <link name="accessories">
-        <visual>
-            <origin rpy="0 0 0" xyz="${body_center_x} ${body_center_y} ${body_center_z}"/>
-            <geometry>
-                <mesh filename="package://legged_unitree_description/meshes/a1/body/textured/accessories.dae" scale="1 1 1"/>
-            </geometry>
-            <material name="blue"/>
-        </visual>
-    </link>
-    <joint name="d435_joint" type="fixed">
-        <parent link="base"/>
-        <child link="d435"/>
-        <origin rpy="0 0 0" xyz="0 0 0"/>
-    </joint>
-    <link name="d435">
-        <visual>
-            <origin rpy="0 0 0" xyz="${body_center_x} ${body_center_y+0.003} ${body_center_z}"/>
-            <geometry>
-                <mesh filename="package://legged_unitree_description/meshes/a1/body/textured/ylo2_d435_textured.dae" scale="1 1 1"/>
-            </geometry>
-            <material name="black"/>
-        </visual>
-    </link>
-    <joint name="t265_joint" type="fixed">
-        <parent link="base"/>
-        <child link="t265"/>
-        <origin rpy="0 0 0" xyz="0 0 0"/>
-    </joint>
-    <link name="t265">
-        <visual>
-            <origin rpy="0 0 0" xyz="${body_center_x} ${body_center_y} ${body_center_z}"/>
-            <geometry>
-                <mesh filename="package://legged_unitree_description/meshes/a1/body/textured/ylo2_t265_textured.dae" scale="1 1.06 1.04"/>
-            </geometry>
-            <material name="black"/>
-        </visual>
-    </link>
     <xacro:IMU connected_to="base" imu_name="unitree_imu" xyz="0. 0. 0." rpy="0. 0. 0."/>
     <xacro:leg prefix="RF" mirror="-1" mirror_dae="False" front_hind="1" front_hind_dae="True">
-        <origin rpy="0 0 0" xyz="${leg_offset_x+0.0345} ${-leg_offset_y+0.005} ${leg_offset_z}"/>
+        <origin rpy="0 0 0" xyz="${leg_offset_x} ${-leg_offset_y} 0"/>
     </xacro:leg>
     <xacro:leg prefix="LF" mirror="1" mirror_dae="True" front_hind="1" front_hind_dae="True">
-        <origin rpy="0 0 0" xyz="${leg_offset_x+0.0345} ${leg_offset_y+0.006} ${leg_offset_z}"/>
+        <origin rpy="0 0 0" xyz="${leg_offset_x} ${leg_offset_y} 0"/>
     </xacro:leg>
     <xacro:leg prefix="RH" mirror="-1" mirror_dae="False" front_hind="-1" front_hind_dae="False">
-        <origin rpy="0 0 0" xyz="${-leg_offset_x-0.0745} ${-leg_offset_y+0.005} ${leg_offset_z}"/>
+        <origin rpy="0 0 0" xyz="${-leg_offset_x} ${-leg_offset_y} 0"/>
     </xacro:leg>
     <xacro:leg prefix="LH" mirror="1" mirror_dae="True" front_hind="-1" front_hind_dae="False">
-        <origin rpy="0 0 0" xyz="${-leg_offset_x-0.0745} ${leg_offset_y+0.006} ${leg_offset_z}"/>
+        <origin rpy="0 0 0" xyz="${-leg_offset_x} ${leg_offset_y} 0"/>
     </xacro:leg>
 </robot>
