Commit message: modified collisions parts

File: legged_ylo2/legged_ylo2_description/urdf/common/leg.xacro (robot description, xacro)
@@ -71,12 +71,7 @@
             </visual>
             <collision>
-                <origin rpy="0 0 0" xyz="0 ${(0.075*mirror)} 0"/>
+                <origin rpy="0 ${pi/2.0+0.05} 0" xyz="0 ${0.074*mirror} -0.07"/>
                 <geometry>
-                    <xacro:if value="${mirror_dae == True}">
-                        <mesh filename="package://legged_ylo2_description/meshes/leg/ylo2_upper_leg_collision.dae" scale="-1 1 1"/>
-                    </xacro:if>
-                    <xacro:if value="${mirror_dae == False}">
-                        <mesh filename="package://legged_ylo2_description/meshes/leg/ylo2_upper_leg_collision.dae" scale="-1 1 1"/>
-                    </xacro:if>
+                    <box size="0.201 0.0374 0.03"/>
                 </geometry>
             </collision>
@@ -111,7 +106,7 @@
             </visual>
             <collision>
-                <origin rpy="0 0 0" xyz="0 0 0"/>
+                <origin rpy="0 ${(pi/2.0-0.1)} 0" xyz="0 0 -0.08"/>
                 <geometry>
-                    <mesh filename="package://legged_ylo2_description/meshes/leg/ylo2_lower_leg_collision.dae" scale="-1 1 1"/>
+                    <box size="0.19 0.02 0.02"/>
                 </geometry>
             </collision>
@@ -140,5 +135,5 @@
         <link name="${prefix}_FOOT">
             <visual>
-                <origin rpy="0 0 0" xyz="0.009 ${(0.001*mirror)+0.001} 0.069"/>
+                <origin rpy="0 0 0" xyz="0.010 ${(0.001*mirror)} 0.069"/>
                 <geometry>
                     <mesh filename="package://legged_ylo2_description/meshes/leg/fl_foot.dae" scale="1.0 1.0 1.0"/>
@@ -146,7 +141,7 @@
             </visual>
             <collision>
-                <origin rpy="0 0 0" xyz="0.009 ${(0.001*mirror)+0.001} 0.069"/>
+                <origin rpy="0 0 0" xyz="0 0 0.02"/>
                 <geometry>
-                    <mesh filename="package://legged_ylo2_description/meshes/leg/fl_foot.dae" scale="1.0 1.0 1.0"/>
+                    <sphere radius="0.022"/>
                 </geometry>
             </collision>

File: legged_ylo2/legged_ylo2_description/urdf/ylo2.xacro (robot description, xacro)
@@ -17,5 +17,5 @@
             <origin rpy="0 0 0" xyz="-0.02 0.003 0.024"/>
             <geometry>
-                <mesh filename="package://legged_ylo2_description/meshes/body/ylo2_body_collision.dae" scale="1 1 1"/>
+                <box size="0.26 0.18 0.14"/>
             </geometry>
         </collision>

File: legged_ylo2/legged_ylo2_description/urdf/ylo2/const.xacro (robot description, xacro)
@@ -19,5 +19,5 @@
     <xacro:property name="calf_width" value="0.0208"/>
     <xacro:property name="calf_height" value="0.016"/>
-    <xacro:property name="foot_radius" value="0.0265"/>
+    <xacro:property name="foot_radius" value="0.012"/>
     <xacro:property name="stick_radius" value="0.01"/>
     <xacro:property name="stick_length" value="0.2"/>
