Commit message: cleaned and improved files, added a .md file

File: legged_ylo2/legged_ylo2_description/urdf/ylo2.urdf (robot description, URDF)
Before this commit: robot robot, 23 links, 22 joints
Links:
- removed link unitree_imu
- added link ylo2_imu, mass 0.01; visual box size=0.015 0.015 0.004
- link LF_FOOT: geometry collision sphere radius=0.022; visual mesh filename=package://legged_ylo2_description/meshes/leg/fl_foot.dae scale=1.0 1.0 1.0
- link LF_calf: geometry collision box size=0.19 0.02 0.02; visual mesh filename=package://legged_ylo2_description/meshes/leg/textured/lower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 scale=1 1 1
- link LF_thigh: geometry collision box size=0.201 0.0374 0.03; visual mesh filename=package://legged_ylo2_description/meshes/leg/textured/ylo2_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 scale=1 1 1
- link LH_FOOT: geometry collision sphere radius=0.022; visual mesh filename=package://legged_ylo2_description/meshes/leg/fl_foot.dae scale=1.0 1.0 1.0
- link LH_calf: geometry collision box size=0.19 0.02 0.02; visual mesh filename=package://legged_ylo2_description/meshes/leg/textured/lower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 scale=1 1 1
- link LH_thigh: geometry collision box size=0.201 0.0374 0.03; visual mesh filename=package://legged_ylo2_description/meshes/leg/textured/ylo2_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 scale=1 1 1
- link RF_FOOT: geometry collision sphere radius=0.022; visual mesh filename=package://legged_ylo2_description/meshes/leg/fl_foot.dae scale=1.0 1.0 1.0
- link RF_calf: geometry collision box size=0.19 0.02 0.02; visual mesh filename=package://legged_ylo2_description/meshes/leg/textured/lower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 scale=1 1 1
- link RF_thigh: geometry collision box size=0.201 0.0374 0.03; visual mesh filename=package://legged_ylo2_description/meshes/leg/textured/ylo2_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 scale=1 -1 1
- link RH_FOOT: geometry collision sphere radius=0.022; visual mesh filename=package://legged_ylo2_description/meshes/leg/fl_foot.dae scale=1.0 1.0 1.0
- link RH_calf: geometry collision box size=0.19 0.02 0.02; visual mesh filename=package://legged_ylo2_description/meshes/leg/textured/lower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 scale=1 1 1
- link RH_thigh: geometry collision box size=0.201 0.0374 0.03; visual mesh filename=package://legged_ylo2_description/meshes/leg/textured/ylo2_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 scale=1 -1 1
- link base: geometry collision box size=0.26 0.18 0.14; visual mesh filename=package://legged_ylo2_description/meshes/body/textured/ylo2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 scale=1 1 1
Joints:
- removed joint unitree_imu_joint
- added joint ylo2_imu_joint: type fixed, parent base, child ylo2_imu, origin xyz=0. 0. 0. rpy=0. 0. 0.

File: legged_ylo2/legged_ylo2_description/urdf/ylo2.xacro (robot description, xacro)
@@ -129,5 +129,5 @@
         <origin rpy="0 0 0" xyz="0 0 0"/>
     </joint>
-    <xacro:IMU connected_to="base" imu_name="unitree_imu" xyz="0. 0. 0." rpy="0. 0. 0."/>
+    <xacro:IMU connected_to="base" imu_name="ylo2_imu" xyz="0. 0. 0." rpy="0. 0. 0."/>
     <xacro:leg prefix="RF" mirror="-1" mirror_dae="False" front_hind="1" front_hind_dae="True">
         <origin rpy="0 0 0" xyz="${leg_offset_x+0.0345} ${-leg_offset_y+0.005} ${leg_offset_z}"/>
